File: PCB/sch.kicad_pcb (KiCad board)
At the start: 2 copper layers, 16 parts, among them J1 PROTON_CONN_LEFT, J2 PROTON_CONN_RIGHT, J3 DISPLAY_CONN

Commit message: SCH Done
Parts:
- added C1: 100uF, Capacitor_SMD:C_0201_0603Metric_Pad0.64x0.40mm_HandSolder, F.Cu at (108.1, 84.2)
- added C2: 100n, Capacitor_SMD:C_0201_0603Metric_Pad0.64x0.40mm_HandSolder, F.Cu at (108.1, 85.9)
- added C3: 100uF, Capacitor_SMD:C_0201_0603Metric_Pad0.64x0.40mm_HandSolder, F.Cu at (108.1, 87.7)
- added D1: 1N4148W, Diode_SMD:D_SOD-123, F.Cu at (114.5, 32.8)
- added D2: 1N4148W, Diode_SMD:D_SOD-123, F.Cu at (114.5, 36.1)
- added J4: TFT_CONN, Connector_PinSocket_2.54mm:PinSocket_1x09_P2.54mm_Vertical, F.Cu at (159.3, 38.1)
- added J5: SD_CONN, Connector_PinSocket_2.54mm:PinSocket_1x05_P2.54mm_Vertical, F.Cu at (127.0, 33.0)
- added J6: GPS_CONN, Connector_PinSocket_2.54mm:PinSocket_1x04_P2.54mm_Vertical, F.Cu at (99.8, 85.6)
- added J7: DEBUG_CONN_L, Connector_PinSocket_2.54mm:PinSocket_1x03_P2.54mm_Vertical, F.Cu at (50.8, 111.8)
- added J8: DEBUG_CONN_R, Connector_PinSocket_2.54mm:PinSocket_1x04_P2.54mm_Vertical, F.Cu at (68.6, 109.2)
- added LS1: Speaker, Connector:CONN_2PIN_SCREW, F.Cu at (112.5, 25.1)
- added Q1: MMBT3904, Package_TO_SOT_SMD:SOT-23, F.Cu at (99.9, 26.6)
- added Q2: MMBT3904, Package_TO_SOT_SMD:SOT-23, F.Cu at (99.9, 31.0)
- added Q3: MMBT3906, Package_TO_SOT_SMD:SOT-23, F.Cu at (99.9, 35.5)
- added Q4: MMBT3906, Package_TO_SOT_SMD:SOT-23, F.Cu at (99.9, 39.9)
- added Q5: MMBT3904, Package_TO_SOT_SMD:SOT-23, F.Cu at (99.9, 44.4)
- added Q6: MMBT3904, Package_TO_SOT_SMD:SOT-23, F.Cu at (99.9, 48.8)
- added R13: 10k, Resistor_SMD:R_0201_0603Metric_Pad0.64x0.40mm_HandSolder, F.Cu at (113.7, 89.4)
- added R14: 470, Resistor_SMD:R_0201_0603Metric_Pad0.64x0.40mm_HandSolder, F.Cu at (113.7, 91.2)
- added R15: 470, Resistor_SMD:R_0201_0603Metric_Pad0.64x0.40mm_HandSolder, F.Cu at (113.7, 92.9)
- added R16: 470, Resistor_SMD:R_0201_0603Metric_Pad0.64x0.40mm_HandSolder, F.Cu at (116.5, 84.2)
- added R17: 470, Resistor_SMD:R_0201_0603Metric_Pad0.64x0.40mm_HandSolder, F.Cu at (116.5, 85.9)
- added R18: 2k2, Resistor_SMD:R_0201_0603Metric_Pad0.64x0.40mm_HandSolder, F.Cu at (116.5, 87.7)
- added R19: 2k2, Resistor_SMD:R_0201_0603Metric_Pad0.64x0.40mm_HandSolder, F.Cu at (116.5, 89.4)
- J3: value DISPLAY_CONN -> KEYPAD_CONN
- R1, R10, R11, R12, R2, R3, R4, R5, R6, R7, R8, R9: footprint Resistor_SMD:R_0805_2012Metric_Pad1.20x1.40mm_HandSolder -> Resistor_SMD:R_0201_0603Metric_Pad0.64x0.40mm_HandSolder
- RV1: footprint Potentiometer_THT:Potentiometer_ACP_CA14-H2,5_Horizontal -> Connector:CONN_3PIN_SCREW
- moved J3 75.7 mm to (39.5, 27.9)
- moved R8 60.4 mm to (42.9, 27.9)
- moved R12 57.8 mm to (35.7, 45.7)
- moved R11 57.6 mm to (35.7, 43.2)
- moved R10 57.4 mm to (35.7, 40.6)
- moved R9 57.1 mm to (35.8, 38.1)
- moved R7 56.2 mm to (42.8, 30.5)
- moved R6 52.3 mm to (42.9, 33.0)
- moved R4 49.6 mm to (42.9, 38.1)
- moved R5 48.7 mm to (42.9, 35.6)
- moved RV1 47.9 mm to (105.5, 76.7)
- moved R3 45.6 mm to (42.9, 40.6)
- moved R2 42.1 mm to (42.9, 43.2)
- moved R1 39.0 mm to (42.9, 45.7)
- moved J1 25.6 mm to (50.8, 25.4)
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Connections:
- J1 pad 1: +5V -> STDIO_UART_HIPO
- J1 pad 2: +3.3V -> KP_ROW_0
- J1 pad 25: unconnected-(J1-Pin_25-Pad25) -> (no net)
- J1 pad 26: unconnected-(J1-Pin_26-Pad26) -> (no net)
- J1 pad 27: unconnected-(J1-Pin_27-Pad27) -> (no net)
- J1 pad 28: unconnected-(J1-Pin_28-Pad28) -> (no net)
- J1 pad 3: GPIO0 -> KP_ROW_1
- J1 pad 4: unconnected-(J1-Pin_4-Pad4) -> KP_ROW_2
- J1 pad 5: unconnected-(J1-Pin_5-Pad5) -> KP_ROW_3
- J1 pad 6: unconnected-(J1-Pin_6-Pad6) -> (no net)
- J1 pad 7: unconnected-(J1-Pin_7-Pad7) -> KP_COL_1
- J1 pad 8: unconnected-(J1-Pin_8-Pad8) -> KP_COL_2
- J1 pad 9: unconnected-(J1-Pin_9-Pad9) -> KP_COL_0
- J2 pad 10: unconnected-(J2-Pin_10-Pad10) -> (no net)
- J2 pad 11: unconnected-(J2-Pin_11-Pad11) -> (no net)
- J2 pad 12: unconnected-(J2-Pin_12-Pad12) -> (no net)
- J2 pad 13: unconnected-(J2-Pin_13-Pad13) -> (no net)
- J2 pad 14: unconnected-(J2-Pin_14-Pad14) -> (no net)
- J2 pad 15: unconnected-(J2-Pin_15-Pad15) -> (no net)
- J2 pad 16: unconnected-(J2-Pin_16-Pad16) -> (no net)
- J2 pad 17: unconnected-(J2-Pin_17-Pad17) -> (no net)
- J2 pad 18: unconnected-(J2-Pin_18-Pad18) -> (no net)
- J2 pad 19: unconnected-(J2-Pin_19-Pad19) -> (no net)
- J2 pad 20: unconnected-(J2-Pin_20-Pad20) -> (no net)
- J2 pad 21: unconnected-(J2-Pin_21-Pad21) -> (no net)
- J2 pad 22: unconnected-(J2-Pin_22-Pad22) -> (no net)
- J2 pad 23: Net-(J2-Pin_23) -> (no net)
- J2 pad 24: unconnected-(J2-Pin_24-Pad24) -> (no net)
- J2 pad 26: unconnected-(J2-Pin_26-Pad26) -> TFT_BACKLIT_LED
- J2 pad 27: +3.3V -> TFT_RST
- J2 pad 28: +5V -> TFT_DC-RS
- J2 pad 7: unconnected-(J2-Pin_7-Pad7) -> (no net)
- J2 pad 8: unconnected-(J2-Pin_8-Pad8) -> (no net)
- J2 pad 9: unconnected-(J2-Pin_9-Pad9) -> (no net)
- R1 pad 1: unconnected-(R1-Pad1) -> KP_COL_1
- R2 pad 1: unconnected-(R2-Pad1) -> KP_COL_2
- R3 pad 1: unconnected-(R3-Pad1) -> KP_COL_3
- R4 pad 1: unconnected-(R4-Pad1) -> KP_COL_0
- R5 pad 1: unconnected-(R5-Pad1) -> KP_ROW_3
- R6 pad 1: unconnected-(R6-Pad1) -> KP_ROW_2
- R7 pad 1: unconnected-(R7-Pad1) -> KP_ROW_1
- R8 pad 1: unconnected-(R8-Pad1) -> KP_ROW_0
- RV1 pad 2: Net-(J2-Pin_23) -> VOL_POT
Routing:
- net GND: track 27.5 -> 0.00 mm
- net Net-(J2-Pin_23): track 10.8 -> 0.00 mm
- net +3.3V: track 9.61 -> 0.00 mm

Commit message: PCB Done
Parts:
- added C4: 100n, Capacitor_SMD:C_0201_0603Metric_Pad0.64x0.40mm_HandSolder, F.Cu at (61.3, 111.4)
- added Q7: MMBT3906, Package_TO_SOT_SMD:SOT-23, B.Cu at (53.6, 70.5)
- added R20: 1k5, Resistor_SMD:R_0201_0603Metric_Pad0.64x0.40mm_HandSolder, B.Cu at (56.8, 74.0)
- added R21: 2K2, Resistor_SMD:R_0201_0603Metric_Pad0.64x0.40mm_HandSolder, F.Cu at (131.4, 59.9)
- added R22: 2K2, Resistor_SMD:R_0201_0603Metric_Pad0.64x0.40mm_HandSolder, F.Cu at (124.9, 60.0)
- C1: footprint Capacitor_SMD:C_0201_0603Metric_Pad0.64x0.40mm_HandSolder -> Capacitor_THT:CP_Radial_D8.0mm_P2.50mm
- C3: value 100uF -> 100n
- moved J3 127.4 mm to (65.1, 152.7), turned to 90 degrees
- moved R9 124.8 mm to (75.2, 156.5), turned to 90 degrees
- moved R10 123.3 mm to (77.8, 156.5), turned to 90 degrees
- moved R8 123.2 mm to (65.1, 149.1), turned to -90 degrees
- moved R11 121.8 mm to (80.3, 156.5), turned to 90 degrees
- moved R7 121.3 mm to (67.6, 149.2), turned to -90 degrees
- moved R12 120.4 mm to (82.9, 156.5), turned to 90 degrees
- moved R6 119.3 mm to (70.2, 149.1), turned to -90 degrees
- moved R5 117.4 mm to (72.7, 149.1), turned to -90 degrees
- moved R4 115.7 mm to (75.2, 149.1), turned to -90 degrees
- moved J4 114.6 mm to (45.7, 52.7)
- moved R3 114.0 mm to (77.8, 149.1), turned to -90 degrees
- moved R2 112.4 mm to (80.3, 149.1), turned to -90 degrees
- moved R1 110.9 mm to (82.9, 149.1), turned to -90 degrees
- moved J1 101.0 mm to (48.9, 126.4), turned to 90 degrees
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Connections:
- C2 pad 1: +3V3 -> +3.3V
- J1 pad 1: STDIO_UART_HIPO -> +5V
- J1 pad 10: unconnected-(J1-Pin_13-Pad10) -> KP_COL_1
- J1 pad 11: unconnected-(J1-Pin_14-Pad11) -> KP_COL_2
- J1 pad 12: unconnected-(J1-Pin_15-Pad12) -> KP_COL_3
- J1 pad 2: KP_ROW_0 -> +3.3V
- J1 pad 25: (no net) -> unconnected-(J1-Pin_25-Pad25)
- J1 pad 26: (no net) -> unconnected-(J1-Pin_26-Pad26)
- J1 pad 27: (no net) -> GPS_UART_HOPI
- J1 pad 28: (no net) -> GND
- J1 pad 3: KP_ROW_1 -> STDIO_UART_HOPI
- J1 pad 4: KP_ROW_2 -> STDIO_UART_HIPO
- J1 pad 5: KP_ROW_3 -> KP_ROW_0
- J1 pad 6: (no net) -> KP_ROW_1
- J1 pad 7: KP_COL_1 -> KP_ROW_2
- J1 pad 8: KP_COL_2 -> KP_ROW_3
- J2 pad 1: (no net) -> +5V
- J2 pad 10: (no net) -> unconnected-(J2-Pin_10-Pad10)
- J2 pad 11: (no net) -> unconnected-(J2-Pin_11-Pad11)
- J2 pad 12: (no net) -> unconnected-(J2-Pin_12-Pad12)
- J2 pad 13: (no net) -> AUD_PWM_B
- J2 pad 14: (no net) -> AUD_PWM_A
- J2 pad 15: (no net) -> SD_SPI_HOPI
- J2 pad 16: (no net) -> SD_SPI_SCK
- J2 pad 17: (no net) -> SD_SPI_CSn
- J2 pad 18: (no net) -> SD_SPI_HIPO
- J2 pad 19: (no net) -> TFT_SPI_HOPI
- J2 pad 2: (no net) -> +3.3V
- J2 pad 20: (no net) -> TFT_SPI_SCK
- J2 pad 21: (no net) -> TFT_SPI_CSn
- J2 pad 22: (no net) -> TFT_DC-RS
- J2 pad 23: (no net) -> TFT_RST
- J2 pad 24: (no net) -> TFT_BACKLIT_LED
- J2 pad 25: unconnected-(J2-Pin_25-Pad25) -> GPS_UART_HIPO
- J2 pad 26: TFT_BACKLIT_LED -> unconnected-(J2-Pin_26-Pad26)
- J2 pad 27: TFT_RST -> unconnected-(J2-Pin_27-Pad27)
- J2 pad 28: TFT_DC-RS -> GND
- J2 pad 3: (no net) -> unconnected-(J2-Pin_3-Pad3)
- J2 pad 4: (no net) -> unconnected-(J2-Pin_4-Pad4)
- J2 pad 5: (no net) -> unconnected-(J2-Pin_5-Pad5)
- J2 pad 6: (no net) -> VOL_POT
- J2 pad 7: (no net) -> unconnected-(J2-Pin_7-Pad7)
- J2 pad 8: (no net) -> unconnected-(J2-Pin_8-Pad8)
- J2 pad 9: (no net) -> unconnected-(J2-Pin_9-Pad9)
- J4 pad 1: +3V3 -> +3.3V
- J4 pad 8: TFT_BACKLIT_LED -> Net-(J4-Pin_8)
- J7 pad 1: (no net) -> STDIO_UART_HIPO
- J7 pad 2: (no net) -> GND
- J7 pad 3: (no net) -> STDIO_UART_HOPI
- J8 pad 1: (no net) -> unconnected-(J8-PBOOT-Pad1)
- J8 pad 2: (no net) -> unconnected-(J8-PSWCLK-Pad2)
- J8 pad 3: (no net) -> GND
- J8 pad 4: (no net) -> unconnected-(J8-PSWD-Pad4)
- Q5 pad 1: AUD_PWM_B -> Net-(Q5-B)
- Q6 pad 1: AUD_PWM_A -> Net-(Q6-B)
- R1 pad 1: KP_COL_1 -> KP_COL_3
- R11 pad 2: Net-(J3-Pin_8) -> Net-(J3-Pin_7)
- R12 pad 2: Net-(J3-Pin_7) -> Net-(J3-Pin_8)
- R13 pad 1: +3V3 -> +3.3V
- R3 pad 1: KP_COL_3 -> KP_COL_1
Routing:
- net +3.3V: track 0.00 -> 267.9 mm, vias 0 -> 2
- net +5V: track 0.00 -> 144.2 mm
- net GND: track 0.00 -> 104.1 mm, vias 0 -> 2
- net AUD_PWM_B: track 0.00 -> 103.4 mm, vias 0 -> 1
- net VOL_POT: track 0.00 -> 96.2 mm, vias 0 -> 1
- net TFT_RST: track 0.00 -> 95.4 mm, vias 0 -> 1
- net TFT_SPI_CSn: track 0.00 -> 93.6 mm, vias 0 -> 1
- net AUD_PWM_A: track 0.00 -> 93.5 mm, vias 0 -> 1
- net TFT_DC-RS: track 0.00 -> 90.7 mm, vias 0 -> 1
- net STDIO_UART_HOPI: track 0.00 -> 89.2 mm
- net TFT_SPI_HOPI: track 0.00 -> 81.7 mm, vias 0 -> 1
- net TFT_SPI_SCK: track 0.00 -> 81.3 mm, vias 0 -> 1
- net STDIO_UART_HIPO: track 0.00 -> 80.8 mm
- net TFT_BACKLIT_LED: track 0.00 -> 72.6 mm, vias 0 -> 1
- net SD_SPI_CSn: track 0.00 -> 59.0 mm
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- added copper zone on F.Cu, net GND
Other:
- board text added: "AUDIO DRIVER"
- board text added: "DISPLAY + SD"
- board text added: "GPS"
- board text added: "KEYPAD"
- board text added: "PROTON BOARD"
- board text added: "TIMEKEEPING"

Commit message: Amended with LDR, Added Gerbers, BOM, positions
Parts:
- added C5: 100n, Capacitor_SMD:C_0201_0603Metric_Pad0.64x0.40mm_HandSolder, F.Cu at (64.1, 111.5)
- added R23: LDR, OptoDevice:R_LDR_5.1x4.3mm_P3.4mm_Vertical, F.Cu at (115.8, 155.7)
- added R24: 10k, Resistor_SMD:R_0201_0603Metric_Pad0.64x0.40mm_HandSolder, F.Cu at (122.0, 155.7)
- R20: value 1k5 -> 510
- moved C2 5.29 mm to (46.1, 50.0), turned to 0 degrees
- moved C4 2.22 mm to (61.2, 113.7)
Connections:
- J2 pad 7: unconnected-(J2-Pin_7-Pad7) -> LDR
Routing:
- net LDR: track 0.00 -> 110.1 mm, vias 0 -> 1
- net +3.3V: track 267.9 -> 291.4 mm
- net GND: track 104.1 -> 101.5 mm
- net SPKR_B: track 23.3 -> 22.3 mm
- net VOL_POT: track 96.2 -> 97.2 mm
- net (no net): track 0.82 -> 0.00 mm
Other:
- board outline added: 107.3 x 120.7 mm
- board text added: "LDR"
- board text added: "VOLUME"
