File: PCB/sch.kicad_sch (KiCad schematic)
At the start: 16 parts, among them J1 PROTON_CONN_LEFT, J2 PROTON_CONN_RIGHT, J3 DISPLAY_CONN

Commit message: SCH Done
Parts:
- added C1, C3: 100uF, Capacitor_SMD:C_0201_0603Metric_Pad0.64x0.40mm_HandSolder, symbol Device:C
- added C2: 100n, Capacitor_SMD:C_0201_0603Metric_Pad0.64x0.40mm_HandSolder, symbol Device:C
- added D1, D2: 1N4148W, Diode_SMD:D_SOD-123, symbol Diode:1N4148W
- added J4: TFT_CONN, Connector_PinSocket_2.54mm:PinSocket_1x09_P2.54mm_Vertical, symbol Connector:Conn_01x09_Socket
- added J5: SD_CONN, Connector_PinSocket_2.54mm:PinSocket_1x05_P2.54mm_Vertical, symbol Connector:Conn_01x05_Socket
- added J6: GPS_CONN, Connector_PinSocket_2.54mm:PinSocket_1x04_P2.54mm_Vertical, symbol Connector:Conn_01x04_Socket
- added J7: DEBUG_CONN_L, Connector_PinSocket_2.54mm:PinSocket_1x03_P2.54mm_Vertical, symbol Connector:Conn_01x03_Socket
- added J8: DEBUG_CONN_R, Connector_PinSocket_2.54mm:PinSocket_1x04_P2.54mm_Vertical, symbol Connector:Conn_01x04_Socket
- added LS1: Speaker, Connector:CONN_2PIN_SCREW, symbol Device:Speaker
- added Q1, Q2, Q5, Q6: MMBT3904, Package_TO_SOT_SMD:SOT-23, symbol Transistor_BJT:MMBT3904
- added Q3, Q4: MMBT3906, Package_TO_SOT_SMD:SOT-23, symbol Transistor_BJT:MMBT3906
- added R13: 10k, Resistor_SMD:R_0201_0603Metric_Pad0.64x0.40mm_HandSolder, symbol Device:R
- added R14, R15, R16, R17: 470, Resistor_SMD:R_0201_0603Metric_Pad0.64x0.40mm_HandSolder, symbol Device:R
- added R18, R19: 2k2, Resistor_SMD:R_0201_0603Metric_Pad0.64x0.40mm_HandSolder, symbol Device:R
- J3: value DISPLAY_CONN -> KEYPAD_CONN
- R1, R10, R11, R12, R2, R3, R4, R5, R6, R7, R8, R9: footprint Resistor_SMD:R_0805_2012Metric_Pad1.20x1.40mm_HandSolder -> Resistor_SMD:R_0201_0603Metric_Pad0.64x0.40mm_HandSolder
- RV1: footprint Potentiometer_THT:Potentiometer_ACP_CA14-H2,5_Horizontal -> Connector:CONN_3PIN_SCREW
Connections:
- net GPIO0 is gone; now on net KP_ROW_1: J1.3 (6)
- net +3.3V: now also J1.3V3 (Pin_2), J2.3V3 (Pin_2), C3.1, J6.1 (Pin_1); no longer J1.2 (Pin_2), J2.27 (Pin_27)
- net +5V: now also J1.5V (Pin_1), J2.5V (Pin_1), C1.1, Q3.2 (E), Q4.2 (E), R18.1, R19.1; no longer J1.1 (Pin_1), J2.28 (Pin_28)
- net GND: now also J1.GND (Pin_28), J2.GND (Pin_28), C1.2, C2.2, C3.2, J4.2 (Pin_2), J6.4 (Pin_4), J7.GND (Pin_2), J8.PGND (Pin_3), Q1.2 (E), Q2.2 (E), Q5.2 (E); no longer J2.29 (Pin_1)
- net KP_ROW_2: now reaches R6.1
- net KP_ROW_2: now also J1.4 (Pin_7)
- net KP_COL_3: now reaches R3.1
- net KP_COL_3: now also J1.9 (Pin_12)
- net KP_COL_0: now reaches R4.1
- net KP_COL_0: now also J1.9 (Pin_12)
- net KP_ROW_3: now reaches R5.1
- net KP_ROW_3: now also J1.5 (Pin_8)
- net VOL_POT: now reaches RV1.2
- net VOL_POT: now also J2.44 (Pin_6); no longer J2.23 (Pin_23)
- net KP_COL_1: now reaches J1.7 (Pin_10)
- net KP_COL_1: now also R1.1
- net KP_COL_2: now reaches J1.8 (Pin_11)
- net KP_COL_2: now also R2.1
- net KP_ROW_1: now reaches R7.1
- net TFT_BACKLIT_LED: now reaches J2.26 (Pin_24)
- net TFT_BACKLIT_LED: now also J4.8 (Pin_8)
- net TFT_SPI_SCK: now reaches J2.30 (Pin_20)
- net TFT_SPI_SCK: now also J4.7 (Pin_7)
- net TFT_SPI_HOPI: now reaches J2.31 (Pin_19)
- net TFT_SPI_HOPI: now also J4.6 (Pin_6)
- net SD_SPI_HIPO: now reaches J2.32 (Pin_18)
- net SD_SPI_HIPO: now also J5.3 (Pin_3), R13.2
- net SD_SPI_CSn: now reaches J2.33 (Pin_17)
- net SD_SPI_CSn: now also J5.1 (Pin_1)
- net SD_SPI_SCK: now reaches J2.34 (Pin_16)
- net SD_SPI_SCK: now also J5.4 (Pin_4)
- net KP_ROW_0: now reaches R8.1
- net KP_ROW_0: now also J1.2 (Pin_5)
- new net: D2.2 (A), Q2.1 (B), R15.1
- new net: Q4.1 (B), R16.2, R19.2
- new net: Q5.3 (C), Q6.2 (E)
- new net: Q3.1 (B), R17.1, R18.2
- new net: D1.2 (A), Q1.1 (B), R14.2
- new net +3V3: C2.1, J4.1 (Pin_1), R13.1
- new net AUD_INH: D1.1 (K), D2.1 (K), Q6.3 (C)
- new net AUD_PWM_A: J2.36 (Pin_14), Q6.1 (B), R14.1
- new net AUD_PWM_B: J2.37 (Pin_13), Q5.1 (B), R15.2
- new net GPS_UART_HIPO: J2.41 (Pin_9), J6.3 (Pin_3)
- new net GPS_UART_HOPI: J2.40 (Pin_10), J6.2 (Pin_2)
- new net SD_SPI_HOPI: J2.35 (Pin_15), J5.2 (Pin_2)
- new net SPKR_A: LS1.1, Q2.3 (C), Q4.3 (C), R17.2
- new net SPKR_B: LS1.2, Q1.3 (C), Q3.3 (C), R16.1
- new net STDIO_UART_HIPO: J1.1 (Pin_4), J7.TX (Pin_1)
- new net STDIO_UART_HOPI: J1.0 (Pin_3), J7.RX (Pin_3)
- new net TFT_DC-RS: J2.28 (Pin_22), J4.5 (Pin_5)
- new net TFT_RST: J2.27 (Pin_23), J4.4 (Pin_4)
- new net TFT_SPI_CSn: J2.29 (Pin_21), J4.3 (Pin_3)
- new net TFT_SPI_HIPO: J4.9 (Pin_9)
- no-connect marks 0 -> 1
Other:
- note added: "AUDIO_DRIVER"
- note added: "DECOUPLING Reduce rail ripple from periodic current draw."
- note added: "DISPLAY_MODULE_INTERFACE"
- note added: "GPS_INTERFACE"
- note added: "H-BRIDGE Drives the Speaker with Vpp = 2 * Vdd or 10V. U := Audio Signal Scaled between 0 and 2*TOP CC_A = ReLU(U - TOP) CC_B = ReLU(TOP - U)"
- note added: "KEYPAD Human Interface for Input- ting Numeric Data. Multi- plex by driving rows high successively and seeing which columns are high, indicating a key press."
- note added: "KEYPAD_INTERFACE"
- note added: "NC"
- note added: "PROTON_BOARD"
- note added: "PROTON_DEBUGGER"
- note added: "SHORT INHIBITOR H-Bridge shorts are prevented in software, but this will limit it to a few ns in case."
- note added: "SPEAKER For our mortal senses!"
- note added: "VOLUME_CONTROL"
- company: (none) -> Kevin Yu
- title: (none) -> LMPK_ALARM_MAIN
- moved on the sheet: J1, J3, R1, R10, R11, R12, R2, R3, R4, R5, R6, R7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

Commit message: PCB Done
Parts:
- added C4: 100n, Capacitor_SMD:C_0201_0603Metric_Pad0.64x0.40mm_HandSolder, symbol Device:C
- added Q7: MMBT3906, Package_TO_SOT_SMD:SOT-23, symbol Transistor_BJT:MMBT3906
- added R20: 1k5, Resistor_SMD:R_0201_0603Metric_Pad0.64x0.40mm_HandSolder, symbol Device:R
- added R21, R22: 2K2, Resistor_SMD:R_0201_0603Metric_Pad0.64x0.40mm_HandSolder, symbol Device:R
- C1: footprint Capacitor_SMD:C_0201_0603Metric_Pad0.64x0.40mm_HandSolder -> Capacitor_THT:CP_Radial_D8.0mm_P2.50mm
- C3: value 100uF -> 100n
- renumbered R12 to R11, R11 to R12
Connections:
- net +3V3 is gone; now on net +3.3V: C2.1, J4.1 (Pin_1), R13.1
- net +3.3V: now also J1.2 (Pin_2), J2.2 (Pin_2), Q7.2 (E); no longer J1.3V3 (Pin_2), J2.3V3 (Pin_2)
- net +5V: now also J1.1 (Pin_1), J2.1 (Pin_1); no longer J1.5V (Pin_1), J2.5V (Pin_1)
- net AUD_PWM_A: now also J2.14 (Pin_14), R22.1; no longer J2.36 (Pin_14), Q6.1 (B)
- net AUD_PWM_B: now also J2.13 (Pin_13), R21.1; no longer J2.37 (Pin_13), Q5.1 (B)
- net GND: now also J1.28 (Pin_28), J2.28 (Pin_28), J7.2 (GND), J8.3 (PGND), C4.1; no longer J1.GND (Pin_28), J2.GND (Pin_28), J7.GND (Pin_2), J8.PGND (Pin_3)
- net GPS_UART_HIPO: now also J2.25 (Pin_25); no longer J2.41 (Pin_9)
- net GPS_UART_HOPI: now also J1.27 (Pin_27); no longer J2.40 (Pin_10)
- net KP_COL_1: now also J1.10 (Pin_10), R3.1; no longer J1.7 (Pin_10), R1.1
- net KP_COL_2: now also J1.11 (Pin_11); no longer J1.8 (Pin_11)
- net KP_COL_3: now also J1.12 (Pin_12), R1.1; no longer J1.9 (Pin_12), R3.1
- net KP_ROW_0: now also J1.5 (Pin_5); no longer J1.2 (Pin_5)
- net KP_ROW_1: now also J1.6 (Pin_6); no longer J1.3 (6)
- net KP_ROW_2: now also J1.7 (Pin_7); no longer J1.4 (Pin_7)
- net KP_ROW_3: now also J1.8 (Pin_8); no longer J1.5 (Pin_8)
- net SD_SPI_CSn: now also J2.17 (Pin_17); no longer J2.33 (Pin_17)
- net SD_SPI_HIPO: now also J2.18 (Pin_18); no longer J2.32 (Pin_18)
- net SD_SPI_HOPI: now also J2.15 (Pin_15); no longer J2.35 (Pin_15)
- net SD_SPI_SCK: now also J2.16 (Pin_16); no longer J2.34 (Pin_16)
- net STDIO_UART_HIPO: now also J1.4 (Pin_4), J7.1 (TX); no longer J1.1 (Pin_4), J7.TX (Pin_1)
- net STDIO_UART_HOPI: now also J1.3 (Pin_3), J7.3 (RX); no longer J1.0 (Pin_3), J7.RX (Pin_3)
- net TFT_BACKLIT_LED: now also J2.24 (Pin_24), R20.2; no longer J2.26 (Pin_24), J4.8 (Pin_8)
- net TFT_DC-RS: now also J2.22 (Pin_22); no longer J2.28 (Pin_22)
- net TFT_RST: now also J2.23 (Pin_23); no longer J2.27 (Pin_23)
- net TFT_SPI_CSn: now also J2.21 (Pin_21); no longer J2.29 (Pin_21)
- net TFT_SPI_HOPI: now also J2.19 (Pin_19); no longer J2.31 (Pin_19)
- net TFT_SPI_SCK: now also J2.20 (Pin_20); no longer J2.30 (Pin_20)
- net VOL_POT: now also J2.6 (Pin_6), C4.2; no longer J2.44 (Pin_6)
- new net: J4.8 (Pin_8), Q7.3 (C)
- new net: Q5.1 (B), R22.2
- new net: Q7.1 (B), R20.1
- new net: Q6.1 (B), R21.2
Other:
- note added: "C4 Smoothens V if pot ends up far from ADC pin"
- moved on the sheet: C2, J4, J5, Q5, Q6, R13, RV1

Commit message: Amended with LDR, Added Gerbers, BOM, positions
Parts:
- added C5: 100nF, Capacitor_SMD:C_0201_0603Metric_Pad0.64x0.40mm, symbol Device:C
- added R23: 10k, OptoDevice:R_LDR_5.1x4.3mm_P3.4mm_Vertical, symbol Device:R
- added R24: 33k, Resistor_SMD:R_0201_0603Metric_Pad0.64x0.40mm, symbol Device:R
- C1: LCSC (none) -> C109392
- C2, C3, C4: value 100n -> 100nF; footprint Capacitor_SMD:C_0201_0603Metric_Pad0.64x0.40mm_HandSolder -> Capacitor_SMD:C_0201_0603Metric_Pad0.64x0.40mm; LCSC (none) -> C14663
- D1, D2: LCSC (none) -> C917030
- LS1, RV1: now left out of the parts list
- Q1, Q2, Q5, Q6: LCSC (none) -> C81464
- Q3, Q4, Q7: LCSC (none) -> C53444
- R1, R2, R3, R4, R5, R6, R7, R8: footprint Resistor_SMD:R_0201_0603Metric_Pad0.64x0.40mm_HandSolder -> Resistor_SMD:R_0201_0603Metric_Pad0.64x0.40mm; LCSC (none) -> C2907002
- R10, R11, R12, R13, R9: footprint Resistor_SMD:R_0201_0603Metric_Pad0.64x0.40mm_HandSolder -> Resistor_SMD:R_0201_0603Metric_Pad0.64x0.40mm; LCSC (none) -> C2906982
- R14, R15, R16, R17: footprint Resistor_SMD:R_0201_0603Metric_Pad0.64x0.40mm_HandSolder -> Resistor_SMD:R_0201_0603Metric_Pad0.64x0.40mm; LCSC (none) -> C23179
- R18, R19: footprint Resistor_SMD:R_0201_0603Metric_Pad0.64x0.40mm_HandSolder -> Resistor_SMD:R_0201_0603Metric_Pad0.64x0.40mm; LCSC (none) -> C2907117
- R20: value 1k5 -> 510; footprint Resistor_SMD:R_0201_0603Metric_Pad0.64x0.40mm_HandSolder -> Resistor_SMD:R_0201_0603Metric_Pad0.64x0.40mm; LCSC (none) -> C2907048
- R21, R22: value 2K2 -> 2k2; footprint Resistor_SMD:R_0201_0603Metric_Pad0.64x0.40mm_HandSolder -> Resistor_SMD:R_0201_0603Metric_Pad0.64x0.40mm; LCSC (none) -> C2907117
Connections:
- net +3.3V: now also R23.1
- net GND: now also C5.2, R24.2
- net LDR: now reaches J2.7 (Pin_7)
- net LDR: now also C5.1, R23.2, R24.1
Other:
- note added: "AMBIENCE_SENSE"
- note added: "BACKLIGHT PWM Respond to ambient brightness."
- note added: "DISPLAY GUI for alarms, pictures, map, and other functions."
- note added: "Read in UTC Time via UART reports, calcu- late US time zone via coordinates."
- note added: "Record Room Brightness with LDR or phototranstor, adjust display brightness with PWM."
- note added: "SD CARD Store music and images and nonvolatile data like UI state, user settings, set alarms."
- note added: "The one and only, by Niraj"
- moved on the sheet: C3, J6
